File: PCB/dombyra.kicad_pcb (KiCad board)
At the start: 2 copper layers, 729 x 124.5 mm, 73 parts, among them J1 Conn_01x04_Socket, J2 Conn_01x04_Socket, J3 USB_C_Receptacle_PowerOnly_6P, U1 ESP32-DEVKIT-V1, U2 TP4056-42-ESOP8, U3 MT3608

Commit message: demo
Parts:
- BT1: footprint Connector_PinHeader_2.00mm:PinHeader_1x02_P2.00mm_Vertical -> Connector_PinHeader_2.54mm:PinHeader_1x02_P2.54mm_Vertical
- C1, C2: footprint Capacitor_THT:CP_Radial_D5.0mm_P2.00mm -> Capacitor_SMD:C_0805_2012Metric
- C3, C4: footprint Capacitor_THT:CP_Radial_D5.0mm_P2.00mm -> Capacitor_SMD:C_1206_3216Metric
- D40: footprint LED_THT:LED_D3.0mm -> LED_THT:LED_D5.0mm
- D41: footprint Diode_SMD:D_SMA -> footprint:SMA_L4.3-W2.6-LS5.2-RD
- L4.7uH1: footprint Inductor_SMD:L_Changjiang_FXL0630 -> Inductor_SMD:L_1812_4532Metric
- R1, R2, R9: footprint Resistor_THT:R_Axial_DIN0204_L3.6mm_D1.6mm_P1.90mm_Vertical -> Resistor_SMD:R_0402_1005Metric
- R10, R3, R4, R5.6k1, R68k1: footprint Resistor_THT:R_Axial_DIN0204_L3.6mm_D1.6mm_P1.90mm_Vertical -> Resistor_SMD:R_0603_1608Metric
- R1k1, R1k2: footprint Resistor_THT:R_Axial_DIN0204_L3.6mm_D1.6mm_P1.90mm_Vertical -> Resistor_SMD:R_0805_2012Metric
- TH1: footprint Library:TRES_MF52-A_CTM -> Connector_PinHeader_2.00mm:PinHeader_2x01_P2.00mm_Vertical
- moved C1 344.3 mm to (392.4, 123.1)
- moved R1k1 343.3 mm to (392.5, 129.8)
- moved R1k2 343.3 mm to (397.3, 138.0)
- moved D40 343.3 mm to (392.8, 143.3)
- moved H6 343.3 mm to (404.1, 154.5)
- moved H7 343.3 mm to (404.1, 93.7)
- moved R2.4k1 343.3 mm to (383.9, 138.4)
- moved R6 343.3 mm to (386.7, 144.8)
- moved U2 343.3 mm to (386.2, 133.3)
- moved D41 343.3 mm to (375.2, 84.5)
- moved H5 343.3 mm to (342.4, 154.5)
- moved H8 343.3 mm to (342.4, 93.7)
- moved J1 343.3 mm to (401.2, 80.2)
- moved U1 343.3 mm to (356.4, 126.2)
- moved D39 343.3 mm to (396.3, 130.5)
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Routing:
- net GND: track 937.5 -> 959.1 mm
- net +5V: track 1136.4 -> 1131.1 mm, vias 3 -> 2
- net Net-(D40-K): track 9.67 -> 10.9 mm
- net Net-(D39-A): track 70.8 -> 72.0 mm
- net Net-(D41-A): track 26.4 -> 27.3 mm
- net Net-(U3-FB): track 23.3 -> 23.8 mm, vias 1 -> 2
- net Net-(BT1-+): track 69.1 -> 69.5 mm, vias 2 -> 3
- net Net-(U1-D22): track 27.4 -> 27.6 mm, vias 0 -> 1
- net Net-(U1-D23): track 35.4 -> 35.6 mm, vias 0 -> 1
- net Net-(U2-~{CHRG}): track 5.38 -> 5.43 mm, vias 1 -> 2
- net Net-(U2-~{STDBY}): vias 1 -> 2
Other:
- board size 729 x 124.5 mm -> 466.1 x 138.7 mm
