File: PCB/dombyra.kicad_sch (KiCad schematic)
At the start: 73 parts, among them J1 Conn_01x04_Socket, J2 Conn_01x04_Socket, J3 USB_C_Receptacle_PowerOnly_6P, U1 ESP32-DEVKIT-V1, U2 TP4056-42-ESOP8, U3 MT3608

Commit message: demo
Parts:
- added U4: SK6812_C5378720, footprint:LED-SMD_4P-L5.4-W5.0_SK6812, symbol SK6812_C5378720:SK6812_C5378720
- BT1: footprint Connector_PinHeader_2.00mm:PinHeader_1x02_P2.00mm_Vertical -> Connector_PinHeader_2.54mm:PinHeader_1x02_P2.54mm_Vertical
- C1, C2: footprint Capacitor_THT:CP_Radial_D5.0mm_P2.00mm -> Capacitor_SMD:C_0805_2012Metric
- C3, C4: footprint Capacitor_THT:CP_Radial_D5.0mm_P2.00mm -> Capacitor_SMD:C_1206_3216Metric
- D40: footprint LED_THT:LED_D3.0mm -> LED_THT:LED_D5.0mm
- D41: footprint Diode_SMD:D_SMA -> footprint:SMA_L4.3-W2.6-LS5.2-RD
- L4.7uH1: footprint Inductor_SMD:L_Changjiang_FXL0630 -> Inductor_SMD:L_1812_4532Metric
- R1, R2, R9: footprint Resistor_THT:R_Axial_DIN0204_L3.6mm_D1.6mm_P1.90mm_Vertical -> Resistor_SMD:R_0402_1005Metric
- R10, R3, R4, R5.6k1, R68k1: footprint Resistor_THT:R_Axial_DIN0204_L3.6mm_D1.6mm_P1.90mm_Vertical -> Resistor_SMD:R_0603_1608Metric
- R1k1, R1k2: footprint Resistor_THT:R_Axial_DIN0204_L3.6mm_D1.6mm_P1.90mm_Vertical -> Resistor_SMD:R_0805_2012Metric
- TH1: footprint Library:TRES_MF52-A_CTM -> Connector_PinHeader_2.00mm:PinHeader_2x01_P2.00mm_Vertical
